File: hardware/controller-f407/rotor_drive.kicad_sch (KiCad schematic)
At the start: 111 parts, among them J1 CDE_1to8, J2 AC_PIGTAIL, K1 G5LE-1A4-DC5, Q1 AO3400A, Q2 2N7002, Q3 2N7002, Q4 2N7002, Q5 BTA16-600SWRG, Q6 BTA16-600SWRG, Q7 BTA16-600SWRG, U1 TPS3823-33DBVR, U10 74LVC1G08GW, U11 MOC3023SM, U12 MOC3023SM, U13 MOC3023SM, U14 LTV-814S-TA1, U15 LTV-814S-TA1, U16 LTV-814S-TA1, U17 LTV-814S-TA1, U2 SN74LVC14APWR, U3 74LVC1G08GW, U4 74LVC1G08GW, U5 74LVC1G08GW, U6 74LVC1G08GW, U7 74LVC1G08GW, U8 74LVC1G08GW, U9 74LVC1G08GW

Commit message: Layout schematic...that was a lot of work after the AI dropped everything randomly
Connections:
- net AC_BUS: no longer D2.2 (A2)
- net AC_FUSED: now also D2.2 (A2)
- net HOLD_CCW: no longer C61.1, D61.1 (K), R63.1
- net N_BRK_DRV: no longer names the net of Q4.3 (D), U13.2
- net N_BRK_G: no longer names the net of Q7.3 (G), R91.2, R92.1
- net N_BRK_LA: no longer names the net of D72.2 (A), R90.2
- net N_BRK_LK: no longer names the net of D72.1 (K), U13.1
- net N_BRK_OG: no longer names the net of R91.1, U13.6
- net N_BRK_S1: no longer names the net of R94.2, R95.1
- net N_BRK_S2: no longer names the net of R95.2, U16.1
- net N_BRK_SN: no longer names the net of C72.1, R93.2
- net N_CCW_DRV: no longer names the net of Q3.3 (D), U12.2
- net N_CCW_G: no longer names the net of Q6.3 (G), R81.2, R82.1
- net N_CCW_LA: no longer names the net of D71.2 (A), R80.2
- net N_CCW_LK: no longer names the net of D71.1 (K), U12.1
- net N_CCW_OG: no longer names the net of R81.1, U12.6
- net N_CCW_S1: no longer names the net of R84.2, R85.1
- net N_CCW_S2: no longer names the net of R85.2, U15.1
- net N_CCW_SN: no longer names the net of C71.1, R83.2
- net N_COIL: no longer names the net of D8.2 (A), K1.2, Q1.3 (D)
- net N_CW_DRV: no longer names the net of Q2.3 (D), U11.2
- net N_CW_G: no longer names the net of Q5.3 (G), R71.2, R72.1
- net N_CW_LA: no longer names the net of D70.2 (A), R70.2
- net N_CW_LK: no longer names the net of D70.1 (K), U11.1
- net N_CW_OG: no longer names the net of R71.1, U11.6
- net N_CW_S1: no longer names the net of R74.2, R75.1
- net N_CW_S2: no longer names the net of R75.2, U14.1
- net N_CW_SN: no longer names the net of C70.1, R73.2
- net N_HDCCW: no longer names the net of D61.2 (A), R62.2
- net N_HDCW: no longer names the net of D60.2 (A), R60.2
- net ROTOR_RETURN renamed GNDPWR
- new net: C61.1, D61.1 (K), R63.1
Other:
- moved on the sheet: C1, C10, C2, C20, C21, C22, C23, C3, C4, C5, C6, C60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

Commit message: nearly complete schematic for discrete logic version
Connections:
- net AC_FUSED is gone; now on net AC_HOT: D1.2 (A), D2.2 (A2), F1.2, K1.1, R30.1, RV1.1
- net AC_HOT: no longer F1.1, J2.1 (Pin_1)
- net GNDPWR: no longer U2.11, U2.13
- net HOLD_CCW: now also C61.1, D61.1 (K), R63.1
- net CAP_A: no longer names the net of C1.1, C2.1, SJ1.1 (A), SJ3.1 (A)
- net CAP_B: no longer names the net of C1.2, C2.2, SJ2.1 (A), SJ4.1 (A)
- net N_ZC: no longer names the net of R30.2, R31.1
- net N_ZC_LED: no longer names the net of R31.2, U17.1
- new net: F1.1, J2.1 (Pin_1)
- new net ROTOR_RETURN: U2.11, U2.13
Other:
- moved on the sheet: C1, C21, C22, D1, D2, MK1, R30, R31, R32, RV1, SJ1, SJ2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
