File: hardware/controller-f407/rotor_drive.kicad_sch (KiCad schematic)
At the start: 111 parts, among them J1 CDE_1to8, J2 AC_PIGTAIL, K1 G5LE-1A4-DC5, Q1 AO3400A, Q2 2N7002, Q3 2N7002, Q4 2N7002, Q5 BTA16-600SWRG, Q6 BTA16-600SWRG, Q7 BTA16-600SWRG, U1 TPS3823-33DBVR, U10 74LVC1G08GW, U11 MOC3023SM, U12 MOC3023SM, U13 MOC3023SM, U14 LTV-814S-TA1, U15 LTV-814S-TA1, U16 LTV-814S-TA1, U17 LTV-814S-TA1, U2 SN74LVC14APWR, U3 74LVC1G08GW, U4 74LVC1G08GW, U5 74LVC1G08GW, U6 74LVC1G08GW, U7 74LVC1G08GW, U8 74LVC1G08GW, U9 74LVC1G08GW

Commit message: Gate the rotor triacs with ARM_OK only (#10)
* Remove the discrete direction interlock from the rotor drive sheet.

CW_GATE, CCW_GATE, and BRK_GATE now require only ARM_OK. The 74LVC14,
the direction AND gates, and the hold RC are gone. D2 stays on AC_FUSED,
after the fuse and before the relay.

Co-authored-by: Cursor Agent <cursoragent@cursor.com>
Co-authored-by: Jeffrey Millar <wa1hco@users.noreply.github.com>

* Tie the ROTOR_RETURN sheet pin to GNDPWR.

A short wire joins the existing hierarchical label to the ground symbol
on C23, so the parent pin and logic ground are one net. The sheet title
names that net ROTOR_RETURN = GNDPWR.

Co-authored-by: Cursor Agent <cursoragent@cursor.com>
Co-authored-by: Jeffrey Millar <wa1hco@users.noreply.github.com>

---------

Co-authored-by: Cursor Agent <cursoragent@cursor.com>
Co-authored-by: Jeffrey Millar <wa1hco@users.noreply.github.com>
Parts:
- removed C4, C5, C7, C8: 100nF, Capacitor_SMD:C_0603_1608Metric, symbol Device:C
- removed C60, C61: 1uF, Capacitor_SMD:C_0805_2012Metric, symbol Device:C
- removed D60, D61: BAT54, Diode_SMD:D_SOD-123, symbol Device:D
- removed R60, R62: 1k, Resistor_SMD:R_0603_1608Metric, symbol Device:R
- removed R61, R63: 100k, Resistor_SMD:R_0603_1608Metric, symbol Device:R
- removed U2: SN74LVC14APWR, Package_SO:TSSOP-14_4.4x5mm_P0.65mm, symbol 74xx:74HC14
- removed U4, U5, U7, U8: 74LVC1G08GW, Package_TO_SOT_SMD:SOT-353_SC-70-5, symbol 74xGxx:74LVC1G08
Connections:
- net CCW_ARM is gone; now on net ARM_OK: U9.2
- net CCW_TERM is gone; now on net AZ_CCW_EN: U9.1
- net CW_ARM is gone; now on net ARM_OK: U6.2
- net CW_TERM is gone; now on net AZ_CW_EN: U6.1
- no-connect marks 3 -> 1
Other:
- note added: "Interlock, 3.3 V. ARM_OK = ARM_EN AND nRESET. Gates off when ARM_OK is low. CW_GATE = AZ_CW_EN AND ARM_OK. CCW_GATE = AZ_CCW_EN AND ARM_OK. BRK_GATE = AZ_BRAKE_EN AND ARM_OK. Direction lockout is the Drive (ADR 0020)."
- note added: "ROTOR INTERFACE AND AC MOTOR DRIVE (azimuth, AC version) F407 controller, first sheet. MCU pin assignment is deferred. Logic ground is ROTOR_RETURN = GNDPWR (CDE terminal 1). See DESIGN-NOTES.md and ADR 0018. Hierarchical labels leave this sheet for the processor sheet and the power sheet."
- note removed: "Interlock, 3.3 V. CW_GATE = CW_EN AND NOT CCW_EN AND ARM_OK AND NOT HOLD_CCW. ARM_OK = ARM_EN AND nRESET. BRK_GATE = AZ_BRAKE_EN AND ARM_OK. HOLD is about 70-110 ms (1 uF, 100k, 74LVC14). See DESIGN-NOTES.md."
- note removed: "ROTOR INTERFACE AND AC MOTOR DRIVE (azimuth, AC version) F407 controller, first sheet. MCU pin assignment is deferred. Logic ground is ROTOR_RETURN (CDE terminal 1). See DESIGN-NOTES.md and ADR 0018. Hierarchical labels leave this sheet for the processor sheet and the power sheet."
