File: hardware/controller-f407/rotor_drive.kicad_sch (KiCad schematic)
At the start: 111 parts, among them J1 CDE_1to8, J2 AC_PIGTAIL, K1 G5LE-1A4-DC5, Q1 AO3400A, Q2 2N7002, Q3 2N7002, Q4 2N7002, Q5 BTA16-600SWRG, Q6 BTA16-600SWRG, Q7 BTA16-600SWRG, U1 TPS3823-33DBVR, U10 74LVC1G08GW, U11 MOC3023SM, U12 MOC3023SM, U13 MOC3023SM, U14 LTV-814S-TA1, U15 LTV-814S-TA1, U16 LTV-814S-TA1, U17 LTV-814S-TA1, U2 SN74LVC14APWR, U3 74LVC1G08GW, U4 74LVC1G08GW, U5 74LVC1G08GW, U6 74LVC1G08GW, U7 74LVC1G08GW, U8 74LVC1G08GW, U9 74LVC1G08GW

Commit message: Remove the discrete direction interlock from the rotor drive sheet.
CW_GATE, CCW_GATE, and BRK_GATE now require only ARM_OK. The 74LVC14,
the direction AND gates, and the hold RC are gone. D2 stays on AC_FUSED,
after the fuse and before the relay.

Co-authored-by: Cursor Agent <cursoragent@cursor.com>
Co-authored-by: Jeffrey Millar <wa1hco@users.noreply.github.com>
Parts:
- removed C4, C5, C7, C8: 100nF, Capacitor_SMD:C_0603_1608Metric, symbol Device:C
- removed C60, C61: 1uF, Capacitor_SMD:C_0805_2012Metric, symbol Device:C
- removed D60, D61: BAT54, Diode_SMD:D_SOD-123, symbol Device:D
- removed R60, R62: 1k, Resistor_SMD:R_0603_1608Metric, symbol Device:R
- removed R61, R63: 100k, Resistor_SMD:R_0603_1608Metric, symbol Device:R
- removed U2: SN74LVC14APWR, Package_SO:TSSOP-14_4.4x5mm_P0.65mm, symbol 74xx:74HC14
- removed U4, U5, U7, U8: 74LVC1G08GW, Package_TO_SOT_SMD:SOT-353_SC-70-5, symbol 74xGxx:74LVC1G08
Connections:
- net CCW_ARM is gone; now on net ARM_OK: U9.2
- net CCW_TERM is gone; now on net AZ_CCW_EN: U9.1
- net CW_ARM is gone; now on net ARM_OK: U6.2
- net CW_TERM is gone; now on net AZ_CW_EN: U6.1
- no-connect marks 3 -> 1
Other:
- note added: "Interlock, 3.3 V. ARM_OK = ARM_EN AND nRESET. Gates off when ARM_OK is low. CW_GATE = AZ_CW_EN AND ARM_OK. CCW_GATE = AZ_CCW_EN AND ARM_OK. BRK_GATE = AZ_BRAKE_EN AND ARM_OK. Direction lockout is the Drive (ADR 0020)."
- note removed: "Interlock, 3.3 V. CW_GATE = CW_EN AND NOT CCW_EN AND ARM_OK AND NOT HOLD_CCW. ARM_OK = ARM_EN AND nRESET. BRK_GATE = AZ_BRAKE_EN AND ARM_OK. HOLD is about 70-110 ms (1 uF, 100k, 74LVC14). See DESIGN-NOTES.md."

Commit message: Tie the ROTOR_RETURN sheet pin to GNDPWR.
A short wire joins the existing hierarchical label to the ground symbol
on C23, so the parent pin and logic ground are one net. The sheet title
names that net ROTOR_RETURN = GNDPWR.

Co-authored-by: Cursor Agent <cursoragent@cursor.com>
Co-authored-by: Jeffrey Millar <wa1hco@users.noreply.github.com>
Other:
- note added: "ROTOR INTERFACE AND AC MOTOR DRIVE (azimuth, AC version) F407 controller, first sheet. MCU pin assignment is deferred. Logic ground is ROTOR_RETURN = GNDPWR (CDE terminal 1). See DESIGN-NOTES.md and ADR 0018. Hierarchical labels leave this sheet for the processor sheet and the power sheet."
- note removed: "ROTOR INTERFACE AND AC MOTOR DRIVE (azimuth, AC version) F407 controller, first sheet. MCU pin assignment is deferred. Logic ground is ROTOR_RETURN (CDE terminal 1). See DESIGN-NOTES.md and ADR 0018. Hierarchical labels leave this sheet for the processor sheet and the power sheet."
Changed lines of the file:
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@@
 		)
 	)
-	(text "ROTOR INTERFACE AND AC MOTOR DRIVE  (azimuth, AC version)\nF407 controller, first sheet. MCU pin assignment is deferred.\nLogic ground is ROTOR_RETURN (CDE terminal 1). See DESIGN-NOTES.md and ADR 0018.\nHierarchical labels leave this sheet for the processor sheet and the power sheet."
+	(text "ROTOR INTERFACE AND AC MOTOR DRIVE  (azimuth, AC version)\nF407 controller, first sheet. MCU pin assignment is deferred.\nLogic ground is ROTOR_RETURN = GNDPWR (CDE terminal 1). See DESIGN-NOTES.md and ADR 0018.\nHierarchical labels leave this sheet for the processor sheet and the power sheet."
 		(exclude_from_sim no)
 		(at 14.986 -39.624 0)
@@
 		)
 	)
+	(wire
+		(pts
+			(xy 137.16 36.83) (xy 121.92 36.83)
+		)
+		(stroke
+			(width 0)
+			(type default)
+		)
+	)
+	(wire
+		(pts
+			(xy 121.92 36.83) (xy 121.92 33.02)
+		)
+		(stroke
+			(width 0)
+			(type default)
+		)
+	)

Commit message: Drive the rotor gates from the MCU and clamp only the relay.
Remove the remaining AND gates so the Drive pins switch the triacs and the relay FET, with pulldowns holding a high-Z pin off. Keep the TPS3823 as a hard clamp on the relay gate. Record the STM32G431 brownout, reset, and option-byte findings in ADR 0021.

Co-authored-by: Jeffrey Millar <wa1hco@users.noreply.github.com>
Co-authored-by: Cursor Agent <cursoragent@cursor.com>
Parts:
- removed C10, C3, C6, C9: 100nF, Capacitor_SMD:C_0603_1608Metric, symbol Device:C
- removed U10, U3, U6, U9: 74LVC1G08GW, Package_TO_SOT_SMD:SOT-353_SC-70-5, symbol 74xGxx:74LVC1G08
- added Q8: MMBT3904, Package_TO_SOT_SMD:SOT-23, symbol Transistor_BJT:MMBT3904
- added Q9: 2N7002, Package_TO_SOT_SMD:SOT-23, symbol Transistor_FET:2N7002
- added R54: 1k, Resistor_SMD:R_0603_1608Metric, symbol Device:R
- added R55: 10k, Resistor_SMD:R_0603_1608Metric, symbol Device:R
- added R56: 100k, Resistor_SMD:R_0603_1608Metric, symbol Device:R
Connections:
- net BRK_GATE is gone; now on net AZ_BRAKE_EN: Q4.1 (G), R4G.1
- net CCW_GATE is gone; now on net AZ_CCW_EN: Q3.1 (G), R3G.1
- net CW_GATE is gone; now on net AZ_CW_EN: Q2.1 (G), R2G.1
- net +3V3: now also R56.1
- net ARM_EN: now also R54.1
- net GNDPWR: now also Q8.2 (E), Q9.2 (S)
- net nRESET: now also R55.1
- net ARM_OK renamed RELAY_GATE
- net RELAY_GATE: now also Q9.3 (D), R54.2
- new net: Q8.1 (B), R55.2
- new net: Q8.3 (C), Q9.1 (G), R56.2
Other:
- note added: "Drive pins, 3.3 V. A pulldown holds each gate off while the pin is high-Z. CW_GATE follows AZ_CW_EN. CCW_GATE follows AZ_CCW_EN. BRK_GATE follows AZ_BRAKE_EN. The relay FET follows ARM_EN. Q9 clamps it off while nRESET is low (ADR 0021)."
- note removed: "Interlock, 3.3 V. ARM_OK = ARM_EN AND nRESET. Gates off when ARM_OK is low. CW_GATE = AZ_CW_EN AND ARM_OK. CCW_GATE = AZ_CCW_EN AND ARM_OK. BRK_GATE = AZ_BRAKE_EN AND ARM_OK. Direction lockout is the Drive (ADR 0020)."

Commit message: Drop the Drive supervisor and the STOP pin.
The TPS3823, Q8, Q9, and their passives leave the rotor sheet. ARM_EN drives the relay FET, with the pulldowns holding a high-Z gate off. STOP stays a Station command. ADR 0021 is Accepted, including the below-POR check and the case that still fails.

Co-authored-by: Jeffrey Millar <wa1hco@users.noreply.github.com>
Co-authored-by: Cursor Agent <cursoragent@cursor.com>
Parts:
- removed C21: 100nF, Capacitor_SMD:C_0603_1608Metric, symbol Device:C
- removed Q8: MMBT3904, Package_TO_SOT_SMD:SOT-23, symbol Transistor_BJT:MMBT3904
- removed Q9: 2N7002, Package_TO_SOT_SMD:SOT-23, symbol Transistor_FET:2N7002
- removed R41, R42, R56: 100k, Resistor_SMD:R_0603_1608Metric, symbol Device:R
- removed R54: 1k, Resistor_SMD:R_0603_1608Metric, symbol Device:R
- removed R55: 10k, Resistor_SMD:R_0603_1608Metric, symbol Device:R
- removed U1: TPS3823-33DBVR, Package_TO_SOT_SMD:SOT-23-5, symbol controller-f407:TPS3823-33
Connections:
- net RELAY_GATE is gone; now on net ARM_EN: Q1.1 (G), R40.1
Other:
- note added: "Drive pins, 3.3 V. A pulldown holds each gate off while the pin is high-Z. CW follows AZ_CW_EN. CCW follows AZ_CCW_EN. The brake follows AZ_BRAKE_EN. The relay FET follows ARM_EN. Low or high-Z leaves K1 open and the brake engaged."
- note removed: "Drive pins, 3.3 V. A pulldown holds each gate off while the pin is high-Z. CW_GATE follows AZ_CW_EN. CCW_GATE follows AZ_CCW_EN. BRK_GATE follows AZ_BRAKE_EN. The relay FET follows ARM_EN. Q9 clamps it off while nRESET is low (ADR 0021)."
