File: hardware/controller-f407/rotor_drive.kicad_sch (KiCad schematic)
At the start: 94 parts, among them J1 CDE_1to8, J2 AC_PIGTAIL, K1 G5LE-1A4-DC5, Q1 AO3400A, Q2 2N7002, Q3 2N7002, Q4 2N7002, Q5 BTA16-600SWRG, Q6 BTA16-600SWRG, Q7 BTA16-600SWRG, U1 TPS3823-33DBVR, U10 74LVC1G08GW, U11 MOC3023SM, U12 MOC3023SM, U13 MOC3023SM, U14 LTV-814S-TA1, U15 LTV-814S-TA1, U16 LTV-814S-TA1, U17 LTV-814S-TA1, U3 74LVC1G08GW, U6 74LVC1G08GW, U9 74LVC1G08GW

Commit message: minor appearch tweak...before Grok makes big changes
Connections:
- net +3V3: no longer C10.1
- net +5V: now also C10.1
- net BRK_GATE: no longer names the net of Q4.1 (G), R4G.1, U10.4
- net CCW_GATE: no longer names the net of Q3.1 (G), R3G.1, U9.4
- net CW_GATE: no longer names the net of Q2.1 (G), R2G.1, U6.4
Other:
- note added: "Yaesu AC (G-450 class): motor CW (Yaesu 5) on J1-5, motor CCW (Yaesu 4) on J1-6, motor common (Yaesu 6) and pot ground (Yaesu 3) on J1-1, pot REF (Yaesu 1) on J1-3, pot wiper (Yaesu 2) on J1-7. Open SJ1/SJ2, close SJ3/SJ4 so the cap sits across the drive ends. G-5500 and HDR-300 keep the cap in the rotor: leave SJ1-SJ4 open and do not fit C1/C2. HDR-300's pinout is not this 1:1 map. It needs a ca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"
- note removed: "26 VAC inlet, fuse, MOV, half-wave tap, current transformer, ARM relay. Logic stays up when ARM opens."
- note removed: "Each channel, left to right: 180 ohm from +5V, red LED (anode toward the resistor), MOC3023SM, 2N7002 to ROTOR_RETURN. Below: 100 ohm gate, 1k gate-to-MT1, BTA16-600SW, 68 ohm + 0.1 uF X2, LTV-814 stuck-on sense. Triacs stand vertical on the bar, 12.7 mm pitch, lead row near board x 34.4."
- note removed: "Interlock, 3.3 V. ARM_OK = ARM_EN AND nRESET. Gates off when ARM_OK is low. CW_GATE = AZ_CW_EN AND ARM_OK. CCW_GATE = AZ_CCW_EN AND ARM_OK. BRK_GATE = AZ_BRAKE_EN AND ARM_OK. Direction lockout is the Drive (ADR 0020)."
- note removed: "ROTOR INTERFACE AND AC MOTOR DRIVE (azimuth, AC version) F407 controller, first sheet. MCU pin assignment is deferred. Logic ground is ROTOR_RETURN = GNDPWR (CDE terminal 1). See DESIGN-NOTES.md and ADR 0018. Hierarchical labels leave this sheet for the processor sheet and the power sheet."
- note removed: "Yaesu AC (G-450 class): land motor CW (Yaesu 5) on J1-5, motor CCW (Yaesu 4) on J1-6, motor common (Yaesu 6) and pot ground (Yaesu 3) on J1-1, pot REF (Yaesu 1) on J1-3, pot wiper (Yaesu 2) on J1-7. Open SJ1/SJ2, close SJ3/SJ4 so the cap sits across the drive ends. G-5500 and HDR-300 keep the cap in the rotor: leave SJ1-SJ4 open and do not fit C1/C2. HDR-300's pinout is not this 1:1 map. It needs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"
- moved on the sheet: C10, C3, C6, C9, D3, D4, D5, D6, D7, D70, D71, D72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
