File: hardware/controller-f407/rotor_drive.kicad_sch (KiCad schematic)
At the start: 78 parts, among them J1 CDE_1to8, J2 AC_PIGTAIL, K1 G5LE-1A4-DC5, Q1 AO3400A, Q2 2N7002, Q3 2N7002, Q4 2N7002, Q5 BTA16-600SWRG, Q6 BTA16-600SWRG, Q7 BTA16-600SWRG, U11 MOC3023SM, U12 MOC3023SM, U13 MOC3023SM, U14 LTV-814S-TA1, U15 LTV-814S-TA1, U16 LTV-814S-TA1, U17 LTV-814S-TA1

Commit message: Add the Drive MCU and analog sheets, and tidy the triac page (#12)
* Add the Drive MCU and analog sheets, and tidy the triac page.

Tie the dangling ROTOR_RETURN label to GNDPWR, clear overlapping field
text without moving owner-placed parts, and hang drive_mcu and
analog_input off the root. Pin assignment follows ADR 0021.

Co-authored-by: Jeffrey Millar <wa1hco@users.noreply.github.com>
Co-authored-by: Cursor Agent <cursoragent@cursor.com>

* Rename the relay net back to ARM_EN and drop the dangling stub.

The owner's label text is ARM_EN again, in place. One pulldown remains
on each gate line. TR1 conditioning stays on the rotor sheet.

Co-authored-by: Jeffrey Millar <wa1hco@users.noreply.github.com>
Co-authored-by: Cursor Agent <cursoragent@cursor.com>

* Record the 57d43f9 rotor sheet in owner_frozen.json.

The layout tweak did not add or remove text keys. The ARM_EN label and the removed stub keep the same keys. Positions are not stored and nothing is moved.

Co-authored-by: Jeffrey Millar <wa1hco@users.noreply.github.com>

---------

Co-authored-by: Cursor Agent <cursoragent@cursor.com>
Co-authored-by: Jeffrey Millar <wa1hco@users.noreply.github.com>
Connections:
- net AMR_EN renamed ARM_EN
Changed lines of the file:
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@@
-	(wire
-		(pts
-			(xy 224.79 92.71) (xy 224.79 91.44)
-		)
-		(stroke
-			(width 0)
-			(type default)
-		)
-	)
 	(wire
 		(pts
@@
 		)
 	)
-	(hierarchical_label "AMR_EN"
+	(hierarchical_label "ARM_EN"
 		(shape input)
 		(at 224.79 92.71 180)
