File: hardware/controller-f407/rotor_drive.kicad_sch (KiCad schematic)
At the start: 78 parts, among them J1 CDE_1to8, J2 AC_PIGTAIL, K1 G5LE-1A4-DC5, Q1 AO3400A, Q2 2N7002, Q3 2N7002, Q4 2N7002, Q5 BTA16-600SWRG, Q6 BTA16-600SWRG, Q7 BTA16-600SWRG, U11 MOC3023SM, U12 MOC3023SM, U13 MOC3023SM, U14 LTV-814S-TA1, U15 LTV-814S-TA1, U16 LTV-814S-TA1, U17 LTV-814S-TA1

Commit message: edits for clarity after Grok created the sheets...still more work to do.
Parts:
- renumbered C20 to C1, C22 to C2, C23 to C3, C72 to C4, C70 to C5, C1 to C6, C2 to C7, C71 to C8, D20 to D1, D3 to D10, D4 to D11, D7 to D12, D71 to D13, D21 to D2, D1 to D3, D2 to D4, D8 to D5, D72 to D6, D70 to D7, D5 to D8, D6 to D9, J2 to J1, J1 to J2, Q7 to Q2, Q4 to Q3, Q5 to Q4, Q2 to Q5, Q3 to Q7, R21 to R1, R90 to R10, R92 to R11, R94 to R12, R93 to R13, R95 to R14, R96 to R15, R71 to R16, R70 to R17, R72 to R18, R74 to R19, R23 to R2, R73 to R20, R75 to R21, R76 to R22, R81 to R23, R80 to R24, R82 to R25, R84 to R26, R83 to R27, R85 to R28, R86 to R29, R2G to R2G1, R20 to R3, R3G to R3G1, R22 to R4, R4G to R4G1, R32 to R5, R31 to R6, R30 to R7, R40 to R8, R91 to R9, SJ3 to SJ1, SJ1 to SJ2, SJ2 to SJ3, U17 to U1, U13 to U2, U16 to U3, U11 to U4, U14 to U5, U12 to U6, U15 to U7
