File: hardware/controller-f407/drive_mcu.kicad_sch (KiCad schematic)
At the start: 12 parts, among them J10 SWD, J11 UART, U20 STM32G431RBTx

Commit message: edits for clarity after Grok created the sheets...still more work to do.
Parts:
- renumbered C107 to C10, C100 to C11, C101 to C12, C102 to C13, C103 to C14, C104 to C15, C108 to C16, C106 to C9, J10 to J3, J11 to J4, R100 to R30, U20 to U8
