File: hardware/controller-f407/controller-f407.kicad_pcb (KiCad board)
At the start: 2 copper layers, 159 x 99 mm, 122 parts, among them J1 AC_PIGTAIL, J2 CDE_1to8, J3 SWD, J4 UART, J5 EL_POT, K1 G5LE-1A4-DC5, Q1 AO3400A, Q2 BTA16-600SWRG, Q3 2N7002, Q4 BTA16-600SWRG, Q5 2N7002, Q6 BTA16-600SWRG, Q7 2N7002, U1 LTV-814S-TA1, U2 MOC3023SM, U3 LTV-814S-TA1, U4 MOC3023SM, U5 LTV-814S-TA1, U6 MOC3023SM, U7 LTV-814S-TA1, U8 STM32G431RBTx

Commit message: Flip C6 and C7 to the bottom of the controller board.
The two motor-run caps stay on their current holes. Those holes already clear the slot-6 bottom edge strip, and the outline's board coordinates are occupied by the heatsink bar and the parts in front of it. Pads stay through-hole. Fab and courtyard move to the back, and the flat-cap leads bend up into the board so they can be soldered from the top.

Co-authored-by: Jeffrey Millar <wa1hco@users.noreply.github.com>
Parts:
- C6, C7: moved to B.Cu
Other:
- board text added: "BOTTOM (6 mm leads: seat on the board, solder from the top)"
- board text added: "BOTTOM, UPRIGHT, H 15.0 max"
- board text added: "BOTTOM. 41.5x40 face on board; leads exit 41.5x20 face at ~10.2 below PCB,"
- board text added: "BOTTOM: C_MOTOR1 || C_MOTOR2 = 133 uF (CDE 130-156); pad 1-1, 2-2"
- board text added: "BOTTOM: cable tie (2.5 mm) through 2x NPTH 3.2 around the body, or RTV it to the board"
- board text added: "BOTTOM: leads straight up through the board (solder from the top)"
- board text added: "BOTTOM: run 2.5 outboard then bend 90 deg up into the board (r ~1, >=1 mm straight from body)"
- board text removed: "(6 mm leads: no flat mount)"
- board text removed: "41.5x40 face on board; leads exit 41.5x20 face at ~10.2 above PCB,"
- board text removed: "C_MOTOR1 || C_MOTOR2 = 133 uF (CDE 130-156); pad 1-1, 2-2"
- board text removed: "UPRIGHT, H 15.0 max"
- board text removed: "cable tie (2.5 mm) through 2x NPTH 3.2 over body, or RTV the body down"
- board text removed: "leads 1.0 straight down"
- board text removed: "run 2.5 outboard then bend 90 deg down (r ~1, >=1 mm straight from body)"
Changed lines of the file:
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@@
 	)
 	(footprint "controller-f407:C_Rect_KEMET_R60_P37.5_L41.5_W20_H40_Flat"
-		(layer "F.Cu")
+		(layer "B.Cu")
 		(at 259.51 141.06 90)
 		(property "Reference" "C6"
 			(at 0 0 90)
-			(layer "F.SilkS")
+			(layer "B.SilkS")
 			(hide yes)
 			(effects
@@
 					(thickness 0.15)
 				)
+				(justify mirror)
 			)
 		)
 		(property "Value" "100uF"
 			(at 0 0 90)
-			(layer "F.Fab")
+			(layer "B.Fab")
 			(hide yes)
 			(effects
@@
 					(thickness 0.15)
 				)
+				(justify mirror)
 			)
 		)
 		(property "Datasheet" "~"
 			(at 0 0 90)
-			(layer "F.Fab")
+			(layer "B.Fab")
 			(hide yes)
 			(effects
@@
 					(thickness 0.15)
 				)
+				(justify mirror)
 			)
 		)
-		(property "Description" "100 uF 100 VDC/63 VAC, flat, leads bent down. Digi-Key 399-13010-ND. Mouser number not found."
+		(property "Description" "100 uF 100 VDC/63 VAC, flat on the bottom, leads bent up into the board and soldered from the top. Digi-Key 399-13010-ND. Mouser number not found."
 			(at 0 0 90)
-			(layer "F.Fab")
+			(layer "B.Fab")
 			(hide yes)
 			(effects
@@
 					(thickness 0.15)
 				)
+				(justify mirror)
 			)
 		)
@@
 			(at 0 0 90)
 			(unlocked yes)
-			(layer "F.Fab")
+			(layer "B.Fab")
 			(hide yes)
 			(effects
@@
 					(thickness 0.15)
 				)
+				(justify mirror)
 			)
 		)
@@
 			(at 0 0 90)
 			(unlocked yes)
-			(layer "F.Fab")
+			(layer "B.Fab")
 			(hide yes)
 			(effects
@@
 					(thickness 0.15)
 				)
+				(justify mirror)
 			)
 		)
@@
 			(at 0 0 90)
 			(unlocked yes)
-			(layer "F.Fab")
+			(layer "B.Fab")
 			(hide yes)
 			(effects
@@
 					(thickness 0.15)
 				)
+				(justify mirror)
 			)
 		)
@@
 	)
 	(footprint "controller-f407:C_Rect_TDK_B32526T_P37.5_L41.5_W24_H15_Upright"
-		(layer "F.Cu")
+		(layer "B.Cu")
 		(at 259.51 80.06 90)
 		(property "Reference" "C7"
 			(at 0 0 90)
-			(layer "F.SilkS")
+			(layer "B.SilkS")
 			(hide yes)
 			(effects
@@
 					(thickness 0.15)
 				)
+				(justify mirror)
 			)
 		)
 		(property "Value" "33uF"
 			(at 0 0 90)
-			(layer "F.Fab")
+			(layer "B.Fab")
 			(hide yes)
 			(effects
@@
 					(thickness 0.15)
 				)
+				(justify mirror)
 			)
 		)
 		(property "Datasheet" "~"
 			(at 0 0 90)
-			(layer "F.Fab")
+			(layer "B.Fab")
 			(hide yes)
 			(effects
@@
 					(thickness 0.15)
 				)
+				(justify mirror)
 			)
 		)
 		(property "Description" ""
 			(at 0 0 90)
-			(layer "F.Fab")
+			(layer "B.Fab")
 			(hide yes)
 			(effects
@@
 					(thickness 0.15)
 				)
+				(justify mirror)
 			)
 		)
@@
 			(at 0 0 90)
 			(unlocked yes)
-			(layer "F.Fab")
+			(layer "B.Fab")
 			(hide yes)
 			(effects
@@
 					(thickness 0.15)
 				)
+				(justify mirror)
 			)
 		)
@@
 			(at 0 0 90)
 			(unlocked yes)
-			(layer "F.Fab")
+			(layer "B.Fab")
 			(hide yes)
 			(effects
@@
 					(thickness 0.15)
 				)
+				(justify mirror)
 			)
 		)
@@
 			(at 0 0 90)
 			(unlocked yes)
-			(layer "F.Fab")
+			(layer "B.Fab")
 			(hide yes)
 			(effects
@@
 					(thickness 0.15)
 				)
+				(justify mirror)
 			)
 		)
@@
 		)
 		(fill no)
-		(layer "F.CrtYd")
+		(layer "B.CrtYd")
 	)
 	(gr_rect
@@
 		)
 		(fill no)
-		(layer "F.CrtYd")
+		(layer "B.CrtYd")
 	)
 	(gr_circle
@@
 		)
 		(fill no)
-		(layer "F.Fab")
+		(layer "B.Fab")
 	)
 	(gr_rect
@@
 		)
 		(fill no)
-		(layer "F.Fab")
+		(layer "B.Fab")
 	)
 	(gr_line
@@
 			(type default)
 		)
-		(layer "F.Fab")
+		(layer "B.Fab")
 	)
 	(gr_line
@@
 			(type default)
 		)
-		(layer "F.Fab")
+		(layer "B.Fab")
 	)
 	(gr_text "extrusion end"
@@
 		)
 	)
-	(gr_text "41.5x40 face on board; leads exit 41.5x20 face at ~10.2 above PCB,"
+	(gr_text "BOTTOM. 41.5x40 face on board; leads exit 41.5x20 face at ~10.2 below PCB,"
 		(at 229.98 36.69 0)
 		(layer "Cmts.User")
@@
 		)
 	)
-	(gr_text "run 2.5 outboard then bend 90 deg down (r ~1, >=1 mm straight from body)"
+	(gr_text "BOTTOM: run 2.5 outboard then bend 90 deg up into the board (r ~1, >=1 mm straight from body)"
 		(at 229.98 38.49 0)
 		(layer "Cmts.User")
@@
 		)
 	)
-	(gr_text "cable tie (2.5 mm) through 2x NPTH 3.2 over body, or RTV the body down"
+	(gr_text "BOTTOM: cable tie (2.5 mm) through 2x NPTH 3.2 around the body, or RTV it to the board"
 		(at 229.98 40.69 0)
 		(layer "Cmts.User")
@@
 		)
 	)
-	(gr_text "C_MOTOR1 || C_MOTOR2 = 133 uF (CDE 130-156); pad 1-1, 2-2"
+	(gr_text "BOTTOM: C_MOTOR1 || C_MOTOR2 = 133 uF (CDE 130-156); pad 1-1, 2-2"
 		(at 229.98 44.69 0)
 		(layer "Cmts.User")
@@
 		)
 	)
-	(gr_text "UPRIGHT, H 15.0 max"
+	(gr_text "BOTTOM, UPRIGHT, H 15.0 max"
 		(at 265.2 38.34 0)
 		(layer "Cmts.User")
@@
 		)
 	)
-	(gr_text "leads 1.0 straight down"
+	(gr_text "BOTTOM: leads straight up through the board (solder from the top)"
 		(at 265.2 42.34 0)
 		(layer "Cmts.User")
@@
 		)
 	)
-	(gr_text "(6 mm leads: no flat mount)"
+	(gr_text "BOTTOM (6 mm leads: seat on the board, solder from the top)"
 		(at 265.2 44.34 0)
 		(layer "Cmts.User")
@@
 	(gr_text "B32526T1336K000"
 		(at 274.26 80.06 90)
-		(layer "F.Fab")
+		(layer "B.Fab")
 		(effects
 			(font
@@
 				(thickness 0.165)
 			)
+			(justify mirror)
 		)
 	)
 	(gr_text "C_MOTOR2"
 		(at 272.26 80.06 90)
-		(layer "F.Fab")
+		(layer "B.Fab")
 		(effects
 			(font
@@
 				(thickness 0.18)
 			)
+			(justify mirror)
 		)
 	)
 	(gr_text "C_MOTOR1 \nR60EW61005000K 100uF flat, H 20.3"
 		(at 274.26 118.51 90)
-		(layer "F.Fab")
+		(layer "B.Fab")
 		(effects
 			(font
@@
 				(thickness 0.18)
 			)
+			(justify mirror)
 		)
 	)
